Commit message: Fixed Arm Configuration

File: urdf/twelvedof_newBAD.urdf (robot description, URDF)
Before this commit: robot twelvedof_new, 44 links, 43 joints
Links:
- link base_link: geometry visual mesh filename=package://project/meshes/base_link.STL
- link link1: mass 0.3 -> 0.15; geometry visual mesh filename=package://project/meshes/link1.STL
- link link10: mass 0.1 -> 0.15; geometry visual mesh filename=package://project/meshes/link10.STL
- link link11: mass 0.1 -> 0.15; geometry visual mesh filename=package://project/meshes/link11.STL
- link link12: mass 0.1 -> 0.15; geometry visual mesh filename=package://project/meshes/link12.STL
- link link2: mass 0.3 -> 0.15; geometry visual mesh filename=package://project/meshes/link2.STL
- link link3: mass 0.3 -> 0.15; geometry visual mesh filename=package://project/meshes/link3.STL
- link link4: mass 0.2 -> 0.15; geometry visual mesh filename=package://project/meshes/link4.STL
- link link5: mass 0.2 -> 0.15; geometry visual mesh filename=package://project/meshes/link5.STL
- link link6: mass 0.2 -> 0.15; geometry visual mesh filename=package://project/meshes/link6.STL
- link link7: mass 0.2 -> 0.15; geometry visual mesh filename=package://project/meshes/link7.STL
- link link8: mass 0.1 -> 0.15; geometry visual mesh filename=package://project/meshes/link8.STL
- link link9: mass 0.1 -> 0.15; geometry visual mesh filename=package://project/meshes/link9.STL
- link motor1: mass 0.4 -> 2.0
- link motor2: mass 0.4 -> 2.0
- link motor3: mass 0.4 -> 2.0
- link motor9: geometry collision cylinder length=0.1 radius=0.02; visual cylinder length=0.1 radius=0.02
Joints:
- joint final2: origin xyz=0 0.2135 0 rpy=0 -1.5708 0 -> xyz=0 0.3035 0 rpy=0 -1.5708 0
- joint theta1: origin xyz=0 0 0.0499999999999999 rpy=1.5707963267949 0 -3.14159265358979 -> xyz=0 0 0.05 rpy=1.5708 0 0
- joint theta10: origin xyz=0 -0.19 0 rpy=3.14159265358979 0 3.14159265358979 -> xyz=0.035 -0.27 0 rpy=0 0 1.5708
- joint theta11: origin xyz=0 -0.244 0 rpy=-1.5707963267949 0 3.14159265358979 -> xyz=0 -0.354 0 rpy=1.5708 0 3.14159263432665
- joint theta12: origin xyz=0 0 0 rpy=0 1.5707963267949 0 -> xyz=0 0 0 rpy=3.1416 -1.5708 3.1416
- joint theta2: origin xyz=0 0.57 0 rpy=0 -1.5707963267949 0 -> xyz=0 0.57 0 rpy=0 -1.5708 0
- joint theta3: origin xyz=0 0 0.4 rpy=3.14159265358979 0 3.14159265358979 -> xyz=0 0 -0.4 rpy=0 0 3.1416
- joint theta4: origin xyz=0 -0.19 0 rpy=3.14159265358979 0 3.14159265358979 -> xyz=0.015 0.15 0 rpy=3.1416 0 0
- joint theta5: origin xyz=0 -0.244 0 rpy=-1.5707963267949 0 3.14159265358979 -> xyz=0 -0.284 0 rpy=-1.5708 0 3.1416
- joint theta7: axis 0 1 0 -> 0 0 1; origin xyz=0 0.4 0 rpy=1.5707963267949 -1.5707963267949 0 -> xyz=0 0.3785 0 rpy=1.5708 1.5708 0
- joint theta8: axis 1 0 0 -> 0 0 1; origin xyz=0 0.555 0 rpy=0 0 3.14159265358979 -> xyz=0 0 -0.135 rpy=1.5708 -1.5708 3.1416
- joint theta9: axis 1 0 0 -> 0 1 0; origin xyz=0.005 0 -0.4 rpy=-3.14159263868864 0 0 -> xyz=0 0.304 0 rpy=3.1416 1.5708 0
