Commit message: Tuning new arm

File: urdf/twelvedof_newunweighted.urdf (robot description, URDF)
Before this commit: robot twelvedof_new, 44 links, 43 joints
Links:
- link base_link: mass 10 -> None
- link link1: mass 0.1 -> None
- link link10: mass 0.1 -> None
- link link11: mass 0.1 -> None
- link link12: mass 0.1 -> None
- link link2: mass 0.1 -> None
- link link3: mass 0.1 -> None
- link link4: mass 0.1 -> None
- link link5: mass 0.1 -> None
- link link6: mass 0.1 -> None
- link link7: mass 0.1 -> None
- link link8: mass 0.1 -> None
- link link9: mass 0.1 -> None
- link motor1: mass 0.4 -> 2.0
- link motor10: mass 1.0 -> 0.1
- link motor11: mass 1.0 -> 0.1
- link motor12: mass 1.0 -> 0.1
- link motor2: mass 0.4 -> 2.0
- link motor3: mass 0.4 -> 2.0
- link motor4: mass 1.5 -> 1.0
- link motor5: mass 1.5 -> 1.0
- link motor6: mass 1.5 -> 1.0
- link motor7: mass 1.5 -> 0.1
- link motor8: mass 1.0 -> 0.1
- link motor9: mass 1.0 -> 0.1
- link mount10: mass 0.2 -> 0.1
- link mount11: mass 0.2 -> 0.1
- link mount12: mass 0.2 -> 0.1
- link mount6: mass 0.2 -> 0.1
- link mount7: mass 0.2 -> 0.1
- link mount8: mass 0.2 -> 0.1
- link mount9: mass 0.2 -> 0.1
- link sphere2: mass 0.01 -> 0.1
