Commit message: Made arm with better configuration

File: urdf/twelvedof_new.urdf (robot description, URDF)
Before this commit: robot twelvedof, 42 links, 41 joints
Links:
- added link cylinder1, mass 0.01; collision cylinder length=0.1 radius=0.01; visual cylinder length=0.1 radius=0.01
- added link cylinder2, mass 0.1; collision cylinder length=0.1 radius=0.01; visual cylinder length=0.1 radius=0.01
- link base_link: geometry visual mesh filename=package://project/meshes/base_link.STL
- link link1: mass 0.12918 -> 0.15; geometry visual mesh filename=package://project/meshes/link1.STL
- link link10: mass 0.0743981881209823 -> 0.15; geometry visual mesh filename=package://project/meshes/link10.STL
- link link11: mass 0.0099414857849685 -> 0.15; geometry visual mesh filename=package://project/meshes/link11.STL
- link link12: mass 0.0230261093724122 -> 0.15; geometry visual mesh filename=package://project/meshes/link12.STL
- link link2: mass 0.13136 -> 0.15; geometry visual mesh filename=package://project/meshes/link2.STL
- link link3: mass 0.0532676480842889 -> 0.15; geometry visual mesh filename=package://project/meshes/link3.STL
- link link4: mass 0.0532676474780037 -> 0.15; geometry visual mesh filename=package://project/meshes/link4.STL
- link link5: mass 0.00994148578496848 -> 0.15; geometry visual mesh filename=package://project/meshes/link5.STL
- link link6: mass 0.0570027293868964 -> 0.15; geometry visual mesh filename=package://project/meshes/link6.STL
- link link7: mass 0.00994148578496851 -> 0.15; geometry visual mesh filename=package://project/meshes/link7.STL
- link link8: mass 0.0532676474780038 -> 0.15; geometry visual mesh filename=package://project/meshes/link8.STL
- link link9: mass 0.0532676474780037 -> 0.15; geometry visual mesh filename=package://project/meshes/link9.STL
- link motor12: geometry collision cylinder length=0.1 radius=0.011; visual cylinder length=0.1 radius=0.011
- link motor4: geometry collision cylinder length=0.1 radius=0.011; visual cylinder length=0.1 radius=0.011
- link motor7: geometry collision cylinder length=0.1 radius=0.011; visual cylinder length=0.1 radius=0.011
- link motor9: geometry collision cylinder length=0.1 radius=0.02; visual cylinder length=0.1 radius=0.02
- link mount1: geometry collision cylinder length=0.1 radius=0.011; visual cylinder length=0.1 radius=0.011
- link mount10: geometry collision cylinder length=0.1 radius=0.005; visual cylinder length=0.1 radius=0.005
- link mount11: geometry collision cylinder length=0.1 radius=0.005; visual cylinder length=0.1 radius=0.005
- link mount12: geometry collision cylinder length=0.1 radius=0.005; visual cylinder length=0.1 radius=0.005
- link mount2: geometry collision cylinder length=0.1 radius=0.005; visual cylinder length=0.1 radius=0.005
- link mount3: geometry collision cylinder length=0.1 radius=0.005; visual cylinder length=0.1 radius=0.005
- link mount4: geometry collision cylinder length=0.1 radius=0.005; visual cylinder length=0.1 radius=0.005
- link mount5: geometry collision cylinder length=0.1 radius=0.005; visual cylinder length=0.1 radius=0.005
- link mount6: geometry collision cylinder length=0.1 radius=0.005; visual cylinder length=0.1 radius=0.005
- link mount7: geometry collision cylinder length=0.1 radius=0.005; visual cylinder length=0.1 radius=0.005
- link mount8: geometry collision cylinder length=0.1 radius=0.005; visual cylinder length=0.1 radius=0.005
- link mount9: geometry collision cylinder length=0.1 radius=0.005; visual cylinder length=0.1 radius=0.005
- link sphere1: geometry collision sphere radius=0.01; visual sphere radius=0.01
- link sphere2: geometry collision sphere radius=0.01; visual sphere radius=0.01
Joints:
- added joint attach-cylinder1: type fixed, parent tip_elbow, child cylinder1
- added joint attach-cylinder2: type fixed, parent tip_full, child cylinder2
- joint theta1: origin xyz=0 0 0.105 rpy=1.5708 0 0 -> xyz=0 0 0.05 rpy=1.5708 0 0
- joint theta10: origin xyz=0 0.13 0 rpy=3.14159265358979 0 1.5707963267949 -> xyz=0.035 -0.27 0 rpy=0 0 1.5708
- joint theta11: axis 0 0 1 -> 0 1 0; origin xyz=0.17 0 0 rpy=3.14159265358979 0 0 -> xyz=0 -0.354 0 rpy=1.5708 0 3.14159263432665
- joint theta12: axis 1 0 0 -> 0 0 1; origin xyz=0 0 0 rpy=1.5707963267949 0 0 -> xyz=0 0 0 rpy=3.1416 -1.5708 3.1416
- joint theta2: axis 0 1 0 -> 1 0 0; origin xyz=0 0.17 0 rpy=1.5708 1.5708 0 -> xyz=0 0.57 0 rpy=0 -1.5708 0
- joint theta3: origin xyz=0.14 0 0 rpy=0 0 1.5707963267949 -> xyz=0 0 -0.4 rpy=0 0 3.1416
- joint theta4: origin xyz=0 -0.13 0 rpy=0 0 3.14159265358979 -> xyz=0.015 0.15 0 rpy=3.1416 0 0
- joint theta5: axis 0 0 1 -> 0 1 0; origin xyz=0 0.13 0 rpy=0 -1.5707963267949 0 -> xyz=0 -0.284 0 rpy=-1.5708 0 3.1416
- joint theta6: axis 1 0 0 -> 0 0 1; origin xyz=0 0 0 rpy=-3.14159265358979 0 0 -> xyz=0 0 0 rpy=3.1416 -1.5708 0
- joint theta7: axis 1 0 0 -> 0 0 1; origin xyz=0 -0.12 0 rpy=0 0 3.14159265358979 -> xyz=0 0.3785 0 rpy=1.5708 1.5708 0
- joint theta8: axis 1 0 0 -> 0 0 1; origin xyz=0 0 0 rpy=3.14159265358979 1.5707963267949 0 -> xyz=0 0 -0.135 rpy=1.5708 -1.5708 3.1416
- joint theta9: origin xyz=0 -0.13 0 rpy=-3.14159265358978 0 0 -> xyz=0 0.304 0 rpy=3.1416 1.5708 0
- joint worldjoint: origin xyz=0 0 0 rpy=0 0 0 -> xyz=0 0 0 rpy=0 0 1.5708

Commit message: Fixed tip orientations

File: urdf/twelvedof_new.urdf (robot description, URDF)
Before this commit: robot twelvedof, 44 links, 43 joints
Links:
- removed link cylinder1
- removed link sphere1
- added link cylinder, mass 0.01; collision cylinder length=0.1 radius=0.01; visual cylinder length=0.1 radius=0.01
- added link sphere, mass 0.01; collision sphere radius=0.01; visual sphere radius=0.01
Joints:
- removed joint attach-cylinder1
- removed joint attach-sphere1
- added joint attach-cylinder: type fixed, parent tip_elbow, child cylinder
- added joint attach-sphere: type fixed, parent tip_elbow, child sphere
- joint final1: origin xyz=0 0 0 rpy=0 0 0 -> xyz=0 0.2535 0.135 rpy=1.5708 0 -1.5708
- joint final2: origin xyz=0 0 0 rpy=0 0 0 -> xyz=0 0.3035 0 rpy=0 -1.5708 0

Commit message: Made links 9 and 10 longer, removed collisions
Arm now draws properly

File: urdf/twelvedof_new.urdf (robot description, URDF)
Before this commit: robot twelvedof_new, 44 links, 43 joints
Links:
- link base_link: geometry visual mesh filename=package://project/meshes/base_link.STL
- link link1: geometry visual mesh filename=package://project/meshes/link1.STL
- link link10: geometry visual mesh filename=package://project/meshes/link10.STL
- link link11: geometry visual mesh filename=package://project/meshes/link11.STL
- link link12: geometry visual mesh filename=package://project/meshes/link12.STL
- link link2: geometry visual mesh filename=package://project/meshes/link2.STL
- link link3: geometry visual mesh filename=package://project/meshes/link3.STL
- link link4: geometry visual mesh filename=package://project/meshes/link4.STL
- link link5: geometry visual mesh filename=package://project/meshes/link5.STL
- link link6: geometry visual mesh filename=package://project/meshes/link6.STL
- link link7: geometry visual mesh filename=package://project/meshes/link7.STL
- link link8: geometry visual mesh filename=package://project/meshes/link8.STL
- link link9: geometry visual mesh filename=package://project/meshes/link9.STL
Joints:
- joint theta10: origin xyz=0 -0.19 0 rpy=3.14159265358979 0 3.14159265358979 -> xyz=0.005 -0.26 0 rpy=3.14159265358979 0 3.14159265358979
- joint theta11: origin xyz=0 -0.244 0 rpy=-1.5707963267949 0 3.14159265358979 -> xyz=0 -0.314 0 rpy=-1.5707963267949 0 3.14159265358979
- joint theta9: origin xyz=0.005 0 -0.4 rpy=-3.14159263868864 0 0 -> xyz=0 0 -0.4 rpy=-3.14159263868864 0 0

Commit message: Changed arm color, made marks .1m long.

File: urdf/twelvedof_new.urdf (robot description, URDF)
Before this commit: robot twelvedof_new, 44 links, 43 joints
Links:
- link cylinder2: geometry collision cylinder length=0.03 radius=0.01; visual cylinder length=0.03 radius=0.01
Joints:
- joint final1: origin xyz=0 0.2535 0.135 rpy=1.5708 0 -1.5708 -> xyz=0 0.2535 0.1 rpy=1.5708 0 -1.5708
- joint final2: origin xyz=0 0.2135 0 rpy=0 -1.5708 0 -> xyz=0 0.1 0 rpy=0 -1.5708 0

Commit message: Small PID Adjustments

File: urdf/twelvedof_new.urdf (robot description, URDF)
Before this commit: robot twelvedof_new, 44 links, 43 joints
Links:
- link link1: mass 0.3 -> 0.1
- link link2: mass 0.3 -> 0.1
- link link3: mass 0.3 -> 0.1
- link link4: mass 0.2 -> 0.1
- link link5: mass 0.2 -> 0.1
- link link6: mass 0.2 -> 0.1
- link link7: mass 0.2 -> 0.1

Commit message: Fixed Link Lengths

File: urdf/twelvedof_new.urdf (robot description, URDF)
Before this commit: robot twelvedof_new, 44 links, 43 joints
Joints:
- joint final1: origin xyz=0 0.2535 0.1 rpy=1.5708 0 -1.5708 -> xyz=0 0.2 0.1 rpy=1.5708 0 -1.5708
- joint theta1: origin xyz=0 0 0.0499999999999999 rpy=1.5707963267949 0 -3.14159265358979 -> xyz=0 0 0.05 rpy=1.5707963267949 0 -3.14159265358979
- joint theta11: origin xyz=0 -0.314 0 rpy=-1.5707963267949 0 3.14159265358979 -> xyz=-0.000158056929492617 -0.34 0 rpy=-1.5707963267949 0 3.14159265358979
- joint theta2: origin xyz=0 0.57 0 rpy=0 -1.5707963267949 0 -> xyz=0 0.55 0 rpy=0 -1.5707963267949 0
- joint theta4: origin xyz=0 -0.19 0 rpy=3.14159265358979 0 3.14159265358979 -> xyz=0.00999999999999997 -0.156 0 rpy=3.14159265358979 0 3.14159265358979
- joint theta5: origin xyz=0 -0.244 0 rpy=-1.5707963267949 0 3.14159265358979 -> xyz=-0.000158056929492672 -0.244 0 rpy=-1.5707963267949 0 3.14159265358979
- joint theta8: origin xyz=0 0.555 0 rpy=0 0 3.14159265358979 -> xyz=0 0.6 0 rpy=0 0 3.14159265358979
